Commit message: completed total body in basic

File: basic/install/package/share/package/urdf/ro.urdf (robot description, URDF)
Before this commit: robot car, 1 links, 0 joints
Links:
- removed link base
- added link base_footprint
- added link base_link; visual box size=0.6 0.4 0.2
- added link camera; visual cylinder length=0.05 radius=0.1
- added link caster_wheel; visual sphere radius=0.05
- added link l_wheel; visual cylinder length=0.05 radius=0.1
- added link r_wheel; visual cylinder length=0.05 radius=0.1
Joints:
- added joint base_joint: type fixed, parent base_footprint, child base_link, origin xyz=0 0 0.1 rpy=0 0 0
- added joint camera_base: type continuous, parent base_link, child camera, origin xyz=0 0 0.225 rpy=0 0 0
- added joint caster_base: type fixed, parent base_link, child caster_wheel, origin xyz=0.225 0 -0.05 rpy=0 0 0
- added joint lwheel_base: type continuous, parent base_link, child l_wheel, origin xyz=-0.15 0.225 0 rpy=0 0 0, axis 0 1 0
- added joint rwheel_base: type continuous, parent base_link, child r_wheel, origin xyz=-0.15 -0.225 0 rpy=0 0 0, axis 0 1 0

File: basic/src/package/urdf/ro.urdf (robot description, URDF)
Before this commit: robot car, 1 links, 0 joints
Links:
- removed link base
- added link base_footprint
- added link base_link; visual box size=0.6 0.4 0.2
- added link camera; visual cylinder length=0.05 radius=0.1
- added link caster_wheel; visual sphere radius=0.05
- added link l_wheel; visual cylinder length=0.05 radius=0.1
- added link r_wheel; visual cylinder length=0.05 radius=0.1
Joints:
- added joint base_joint: type fixed, parent base_footprint, child base_link, origin xyz=0 0 0.1 rpy=0 0 0
- added joint camera_base: type continuous, parent base_link, child camera, origin xyz=0 0 0.225 rpy=0 0 0
- added joint caster_base: type fixed, parent base_link, child caster_wheel, origin xyz=0.225 0 -0.05 rpy=0 0 0
- added joint lwheel_base: type continuous, parent base_link, child l_wheel, origin xyz=-0.15 0.225 0 rpy=0 0 0, axis 0 1 0
- added joint rwheel_base: type continuous, parent base_link, child r_wheel, origin xyz=-0.15 -0.225 0 rpy=0 0 0, axis 0 1 0
