Commit message: simplerobo simulation in gazebo

File: gbasic/install/package/share/package/urdf/robo.urdf (robot description, URDF)
Before this commit: robot car, 1 links, 0 joints
Links:
- added link base_footprint
- added link caster_wheel, mass 1.0; collision sphere radius=0.05; visual sphere radius=0.05
- added link lidar, mass 1.0; collision cylinder length=0.05 radius=0.1; visual cylinder length=0.05 radius=0.1
- added link wheel_l, mass 1.0; collision cylinder length=0.05 radius=0.1; visual cylinder length=0.05 radius=0.1
- added link wheel_r, mass 1.0; collision cylinder length=0.05 radius=0.1; visual cylinder length=0.05 radius=0.1
- link base_link: mass None -> 1.0
Joints:
- added joint base_joint: type fixed, parent base_footprint, child base_link
- added joint caster_joint: type fixed, parent base_link, child caster_wheel, origin xyz=0.2 0 -0.05 rpy=0 0 0
- added joint left_joint: type continuous, parent base_link, child wheel_l, origin xyz=-0.15 0.225 0 rpy=0 0 0, axis 0 1 0
- added joint lidar_joint: type fixed, parent base_link, child lidar, origin xyz=0 0 0.225 rpy=0 0 0, axis 0 0 0
- added joint right_joint: type continuous, parent base_link, child wheel_r, origin xyz=-0.15 -0.225 0 rpy=0 0 0, axis 0 0 0

Commit message: robot is moving with commands

File: gbasic/install/package/share/package/urdf/robo.urdf (robot description, URDF)
Before this commit: robot car, 6 links, 5 joints
Joints:
- joint right_joint: axis 0 0 0 -> 0 1 0

Commit message: basic model simulation in gzebo

File: gbasic/install/package/share/package/urdf/robo.urdf (robot description, URDF)
Before this commit: robot car, 6 links, 5 joints
Links:
- removed link lidar
- added link lidar_link, mass 1.0; collision cylinder length=0.05 radius=0.1; visual cylinder length=0.05 radius=0.1
Joints:
- joint lidar_joint: child lidar -> lidar_link
